File: WSPRAmp-layout.kicad_pcb (KiCad board)
At the start: 2 copper layers, 101 x 64 mm, 18 parts, among them J1 Conn_Coaxial_Small, J2 Conn_01x05, U3 T2N7002AK_G0_00

Commit message: Update PCB footprints, drill sizes, header previews and silkscreen
Parts:
- R3: footprint Resistor_THT:R_Axial_DIN0614_L14.3mm_D5.7mm_P15.24mm_Horizontal -> Resistor_THT:R_Axial_DIN0309_L9.0mm_D3.2mm_P12.70mm_Horizontal
- RV1: footprint Potentiometer_SMD:Potentiometer_ACP_CA14-VSMD_Vertical -> WSPRAmp:Potentiometer_Trimmer_Horizontal_Triangle_P5.00mm_H5.00mm
- RZ1: footprint Private:RP2040-Zero -> WSPRAmp:RP2040-Zero_Headers_P2.54mm
Routing:
- net Net-(C2-Pad1): track 85.8 -> 91.0 mm
- net Net-(J2-Pin_1): track 52.9 -> 56.6 mm
- net GND: track 7.74 -> 5.04 mm
- net Net-(R1-Pad2): track 41.2 -> 38.7 mm
Other:
- board text added: "RP 2040 Zero WSPR transmitter"
