File: WSPRAmp-layout.kicad_pcb (KiCad board)
At the start: 2 copper layers, 101 x 64 mm, 18 parts, among them J1 Conn_Coaxial_Small, J2 Conn_01x05, U3 T2N7002AK_G0_00

Commit message: Cleaned up old files
Parts:
- J1: footprint Connector_Coaxial:SMA_Amphenol_132289_EdgeMount -> Connector_Coaxial:SMA_Molex_73251-2120_EdgeMount_Horizontal

Commit message: Board fixes for transformer, holes
Parts:
- added H1: MountingHole_2.2mm_M2, MountingHole:MountingHole_2.2mm_M2, F.Cu at (43.5, 37.5)
- added H2: MountingHole_2.2mm_M2, MountingHole:MountingHole_2.2mm_M2, F.Cu at (137.5, 37.5)
- added H3: MountingHole_2.2mm_M2, MountingHole:MountingHole_2.2mm_M2, F.Cu at (43.5, 94.5)
- added H4: MountingHole_2.2mm_M2, MountingHole:MountingHole_2.2mm_M2, F.Cu at (137.5, 94.5)
- moved LS1 15.4 mm to (91.2, 51.1), turned to 180 degrees
- moved J2 5.00 mm to (44.0, 43.0)
Routing:
- net Net-(C4-Pad1): track 12.5 -> 30.0 mm
- net Net-(U3-3): track 27.8 -> 45.0 mm
- net GND: track 5.04 -> 16.0 mm
- net Net-(J2-Pin_1): track 56.6 -> 51.5 mm
- net Net-(J2-Pin_5): track 29.7 -> 24.7 mm
- net Net-(J2-Pin_3): track 28.6 -> 23.6 mm

Commit message: Sumbit to DKRed, etc
Parts:
- J1: footprint Connector_Coaxial:SMA_Molex_73251-2120_EdgeMount_Horizontal -> WSPRAmp:SMA_Edge_6.3mm
- moved J1 0.21 mm to (138.6, 53.0), turned to -90 degrees
