File: WSPRAmp.kicad_sch (KiCad schematic)
At the start: 18 parts, among them J1 Conn_Coaxial_Small, J2 Conn_01x05, U3 T2N7002AK_G0_00

Commit message: Route WSPRAmp board and add upright FT37-43 assemblies
Reserve plug-in GPS space, pair transformer windings on one core, and add local footprints, 3D model, and schematic assignments. Verify zero DRC errors and unconnected items; retain known RP2040 footprint-library warning.
Parts:
- L2: footprint Inductor_THT:L_Axial_L11.0mm_D4.5mm_P15.24mm_Horizontal_Fastron_MECC -> WSPRAmp:FT37-43_Upright_Inductor_P15.24mm
- L3: footprint Inductor_THT:L_Axial_L14.0mm_D4.5mm_P7.62mm_Vertical_Fastron_LACC -> WSPRAmp:FT37-43_Upright_Inductor_P15.24mm
- LP1: footprint Inductor_THT:L_Axial_L11.0mm_D4.5mm_P15.24mm_Horizontal_Fastron_MECC -> WSPRAmp:FT37-43_Upright_Bifilar_Primary
- LS1: footprint Inductor_THT:L_Axial_L11.0mm_D4.5mm_P15.24mm_Horizontal_Fastron_MECC -> WSPRAmp:FT37-43_Upright_Bifilar_Secondary
Changed lines of the file:
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@@
 			)
 		)
-		(property "Footprint" "Inductor_THT:L_Axial_L14.0mm_D4.5mm_P7.62mm_Vertical_Fastron_LACC"
+		(property "Footprint" "WSPRAmp:FT37-43_Upright_Inductor_P15.24mm"
 			(at 207.01 109.22 0)
 			(hide yes)
@@
 			)
 		)
-		(property "Footprint" "Inductor_THT:L_Axial_L11.0mm_D4.5mm_P15.24mm_Horizontal_Fastron_MECC"
+		(property "Footprint" "WSPRAmp:FT37-43_Upright_Bifilar_Secondary"
 			(at 160.02 102.87 0)
 			(hide yes)
@@
 			)
 		)
-		(property "Footprint" "Inductor_THT:L_Axial_L11.0mm_D4.5mm_P15.24mm_Horizontal_Fastron_MECC"
+		(property "Footprint" "WSPRAmp:FT37-43_Upright_Inductor_P15.24mm"
 			(at 199.39 109.22 0)
 			(hide yes)
@@
 			)
 		)
-		(property "Footprint" "Inductor_THT:L_Axial_L11.0mm_D4.5mm_P15.24mm_Horizontal_Fastron_MECC"
+		(property "Footprint" "WSPRAmp:FT37-43_Upright_Bifilar_Primary"
 			(at 149.86 102.87 0)
 			(hide yes)

Commit message: Sync schematic footprints with confirmed PCB packages
Parts:
- J2: footprint Connector_PinHeader_1.27mm:PinHeader_1x05_P1.27mm_Vertical -> Connector_PinHeader_2.54mm:PinHeader_1x05_P2.54mm_Vertical
- L1: footprint Inductor_THT:L_Axial_L14.0mm_D4.5mm_P7.62mm_Vertical_Fastron_LACC -> Inductor_THT:L_Axial_L11.0mm_D4.5mm_P15.24mm_Horizontal_Fastron_MECC
- R1: footprint Resistor_THT:R_Axial_DIN0204_L3.6mm_D1.6mm_P5.08mm_Vertical -> Resistor_THT:R_Axial_DIN0309_L9.0mm_D3.2mm_P12.70mm_Horizontal
Changed lines of the file:
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@@
 			)
 		)
-		(property "Footprint" "Resistor_THT:R_Axial_DIN0204_L3.6mm_D1.6mm_P5.08mm_Vertical"
+		(property "Footprint" "Resistor_THT:R_Axial_DIN0309_L9.0mm_D3.2mm_P12.70mm_Horizontal"
 			(at 101.6 124.46 0)
 			(hide yes)
@@
 			)
 		)
-		(property "Footprint" "Connector_PinHeader_1.27mm:PinHeader_1x05_P1.27mm_Vertical"
+		(property "Footprint" "Connector_PinHeader_2.54mm:PinHeader_1x05_P2.54mm_Vertical"
 			(at 24.13 54.61 0)
 			(hide yes)
@@
 			)
 		)
-		(property "Footprint" "Inductor_THT:L_Axial_L14.0mm_D4.5mm_P7.62mm_Vertical_Fastron_LACC"
+		(property "Footprint" "Inductor_THT:L_Axial_L11.0mm_D4.5mm_P15.24mm_Horizontal_Fastron_MECC"
 			(at 124.46 76.2 0)
 			(hide yes)

Commit message: Update PCB footprints, drill sizes, header previews and silkscreen
Parts:
- R3: footprint Resistor_THT:R_Axial_DIN0614_L14.3mm_D5.7mm_P15.24mm_Horizontal -> Resistor_THT:R_Axial_DIN0309_L9.0mm_D3.2mm_P12.70mm_Horizontal
- RV1: footprint Potentiometer_SMD:Potentiometer_ACP_CA14-VSMD_Vertical -> WSPRAmp:Potentiometer_Trimmer_Horizontal_Triangle_P5.00mm_H5.00mm
- RZ1: footprint Private:RP2040-Zero -> WSPRAmp:RP2040-Zero_Headers_P2.54mm
Changed lines of the file:
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@@
 			)
 		)
-		(property "Footprint" "Potentiometer_SMD:Potentiometer_ACP_CA14-VSMD_Vertical"
+		(property "Footprint" "WSPRAmp:Potentiometer_Trimmer_Horizontal_Triangle_P5.00mm_H5.00mm"
 			(at 86.36 124.46 0)
 			(hide yes)
@@
 			)
 		)
-		(property "Footprint" "Resistor_THT:R_Axial_DIN0614_L14.3mm_D5.7mm_P15.24mm_Horizontal"
+		(property "Footprint" "Resistor_THT:R_Axial_DIN0309_L9.0mm_D3.2mm_P12.70mm_Horizontal"
 			(at 140.97 104.14 0)
 			(hide yes)
@@
 			)
 		)
-		(property "Footprint" "Private:RP2040-Zero"
+		(property "Footprint" "WSPRAmp:RP2040-Zero_Headers_P2.54mm"
 			(at 35.1633 127 0)
 			(show_name no)
