File: WSPRAmp-layout.kicad_sch (KiCad schematic)
At the start: 18 parts, among them J1 Conn_Coaxial_Small, J2 Conn_01x05, U3 T2N7002AK_G0_00

Commit message: Board fixes for transformer, holes
Parts:
- J1: footprint Connector_Coaxial:SMA_Amphenol_132289_EdgeMount -> Connector_Coaxial:SMA_Molex_73251-2120_EdgeMount_Horizontal
Changed lines of the file:
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@@
 			)
 		)
-		(property "Footprint" "Connector_Coaxial:SMA_Amphenol_132289_EdgeMount"
+		(property "Footprint" "Connector_Coaxial:SMA_Molex_73251-2120_EdgeMount_Horizontal"
 			(at 223.52 110.49 0)
 			(hide yes)

Commit message: Sumbit to DKRed, etc
Parts:
- J1: footprint Connector_Coaxial:SMA_Molex_73251-2120_EdgeMount_Horizontal -> WSPRAmp:SMA_Edge_6.3mm
Changed lines of the file:
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@@
 			)
 		)
-		(property "Footprint" "Connector_Coaxial:SMA_Molex_73251-2120_EdgeMount_Horizontal"
+		(property "Footprint" "WSPRAmp:SMA_Edge_6.3mm"
 			(at 223.52 110.49 0)
 			(hide yes)
